Commit message: fixed co602 urdf gripper link no found bug

File: hsr_description/urdf/hsr_co602_with_gripper.xacro (robot description, xacro)
@@ -3,4 +3,9 @@
   name="hsr_co602" xmlns:xacro="http://www.ros.org/wiki/xacro">
 <xacro:include filename="$(find hsr_description)/urdf/hsr_co602.urdf" />
+  <joint name="gripper_robot_joint" type="fixed">
+      <parent link="link6" />
+      <child link="gripper_base_link" />
+      <origin xyz="0.0 0.0 0.0" rpy="0 0 0" />
+  </joint>
   <joint name="pick_gripper_joint" type="fixed">
      <origin xyz="-0.0115 0.0 0.15" rpy="0 -1.5708 1.5708" />

File: hsr_description/urdf/hsr_co602_with_gripper_kinect.xacro (robot description, xacro)
@@ -3,4 +3,9 @@
   name="hsr_br606" xmlns:xacro="http://www.ros.org/wiki/xacro">
 <xacro:include filename="$(find hsr_description)/urdf/hsr_co602.urdf" />
+  <joint name="gripper_robot_joint" type="fixed">
+      <parent link="link6" />
+      <child link="gripper_base_link" />
+      <origin xyz="0.0 0.0 0.0" rpy="0 0 0" />
+  </joint>
   <joint name="pick_gripper_joint" type="fixed">
      <origin xyz="-0.0115 0.0 0.15" rpy="0 -1.5708 0" />
