Commit message: jr603分支

File: hsr_description/urdf/hsr_jr603.urdf (robot description, URDF)
Before this commit: robot hsr_jr603, 8 links, 7 joints
Links:
- link base_link: mass 0.00059012 -> 6.73; geometry collision mesh filename=package://hsr_description/meshes/jr603/base_link.STL; visual mesh filename=package://hsr_description/meshes/jr603/base_link.STL
- link link1: mass 0.00059012 -> 2.1859; geometry collision mesh filename=package://hsr_description/meshes/jr603/link1.STL; visual mesh filename=package://hsr_description/meshes/jr603/link1.STL
- link link2: mass 0.00010323 -> 4.4815; geometry collision mesh filename=package://hsr_description/meshes/jr603/link2.STL; visual mesh filename=package://hsr_description/meshes/jr603/link2.STL
- link link3: mass 0.00059012 -> 1.6556; geometry collision mesh filename=package://hsr_description/meshes/jr603/link3.STL; visual mesh filename=package://hsr_description/meshes/jr603/link3.STL
- link link4: mass 0.00059012 -> 1.4831; geometry collision mesh filename=package://hsr_description/meshes/jr603/link4.STL; visual mesh filename=package://hsr_description/meshes/jr603/link4.STL
- link link5: mass 0.00038537 -> 0.37027; geometry collision mesh filename=package://hsr_description/meshes/jr603/link5.STL; visual mesh filename=package://hsr_description/meshes/jr603/link5.STL
- link link6: mass 0.00010153 -> 0.019515; geometry collision mesh filename=package://hsr_description/meshes/jr603/link6.STL; visual mesh filename=package://hsr_description/meshes/jr603/link6.STL
Joints:
- joint joint_1: axis 0 0 -1 -> 0 0 1; limit lower=-3.412119 upper=3.412119 effort=0 velocity=0 -> lower=-3.4819 upper=3.4819 effort=28 velocity=3.2; origin xyz=0 0 0 rpy=-1.0992E-17 -1.7466E-16 -5.4991E-16 -> xyz=0 0 0 rpy=-9.7175E-17 -2.6052E-16 6.9389E-18; type continuous -> revolute
- joint joint_2: limit lower=-3.132866 upper=0 effort=0 velocity=0 -> lower=-2.60926 upper=0.07853 effort=28 velocity=3.2; origin xyz=0 0.0075 0 rpy=-1.5708 6.364E-17 -8.6055E-19 -> xyz=0 0.0075 0 rpy=-1.5708 -1.5582E-16 -7.8704E-17; type continuous -> revolute
- joint joint_3: limit lower=-0.340339 upper=4.180064 effort=0 velocity=0 -> lower=0 upper=4.0927 effort=28 velocity=3.2; origin xyz=0.284 0 -0.0075 rpy=-1.2235E-19 -6.2402E-19 2.3592E-16 -> xyz=0.284 0 -0.0075 rpy=7.2825E-17 -9.1181E-17 9.7145E-17; type continuous -> revolute
- joint joint_4: limit lower=-3.132866 upper=3.132866 effort=0 velocity=0 -> lower=-3.124139 upper=3.124139 effort=28 velocity=3.2; origin xyz=-0.03 0 0 rpy=1.5708 2.8877E-16 7.8886E-31 -> xyz=-0.03 0 0 rpy=1.5708 7.4106E-16 -2.0931E-17; type continuous -> revolute
- joint joint_5: limit lower=-1.998402 upper=1.998402 effort=0 velocity=0 -> lower=-1.562069680534 upper=1.666789435654 effort=28 velocity=3.2; origin xyz=0 0 0.2865 rpy=-1.5708 1.1096E-16 2.8115E-16 -> xyz=0 0 0.2865 rpy=-1.5708 2.0867E-17 -2.541E-17; type continuous -> revolute
- joint joint_6: limit lower=-6.274459 upper=6.274459 effort=0 velocity=0 -> lower=-6.283185307179 upper=6.283185307179 effort=28 velocity=3.2; origin xyz=0 -0.0815 0 rpy=-1.3342 1.5708 -2.905 -> xyz=0 -0.0815 0 rpy=1.5708 -1.5708 0; type continuous -> revolute
