Commit message: 1,add br606 link material 2,add global moveit.rviz 3,change br609 joint type

File: hsr_description/urdf/hsr_br609.urdf (robot description, URDF)
Before this commit: robot hsr_br609, 8 links, 7 joints
Joints:
- joint joint_1: limit (none) -> lower=-2.71415 upper=2.71415 effort=28.0 velocity=3.2; type continuous -> revolute
- joint joint_2: limit (none) -> lower=-3.1 upper=0 effort=28.0 velocity=3.2; type continuous -> revolute
- joint joint_3: limit (none) -> lower=-0.63 upper=3.4 effort=28.0 velocity=3.2; type continuous -> revolute
- joint joint_4: limit (none) -> lower=-1.57 upper=1.57 effort=28.0 velocity=3.2; type continuous -> revolute
- joint joint_5: limit (none) -> lower=-1.68 upper=1.68 effort=28.0 velocity=3.2; type continuous -> revolute
- joint joint_6: limit (none) -> lower=-4.5 upper=4.5 effort=28.0 velocity=3.2; type continuous -> revolute

Commit message: br609的URDF，带夹爪URDF以及相关moveit配置

File: hsr_description/urdf/hsr_br609.urdf (robot description, URDF)
Before this commit: robot hsr_br609, 8 links, 7 joints
Links:
- link base_link: mass 10.953 -> 10.954; geometry collision mesh filename=package://hsr_description/meshes/br609/base_link.STL; visual mesh filename=package://hsr_description/meshes/br609/base_link.STL
- link link1: mass 4.59274863839256 -> 4.6413
- link link2: mass 5.90673615464513 -> 5.9083
- link link3: mass 1.11115703458445 -> 1.1112
- link link4: mass 2.67522980678295 -> 2.67517353862944
- link link5: mass 0.867826372031057 -> 0.868403298162055
- link link6: mass 0.0270769176758969 -> 0.027077
Joints:
- joint fixed: origin (none) -> xyz=0 0 1 rpy=0 0 0
- joint joint_1: axis 0 -1 0 -> 0 0 1; origin xyz=0 0 0.2755 rpy=-1.5708 -6.123E-17 -1.5708 -> xyz=0 0 0 rpy=0 0 0
- joint joint_2: axis 0 0 -1 -> 0 0 1; origin xyz=0 -0.145 0 rpy=-1.5707963267949 -1.22460635382238E-16 1.5707963267949 -> xyz=0 -0.0965 0 rpy=-1.5708 -3.3106E-34 2.6541E-17
- joint joint_3: origin xyz=-0.625999999928 0 -0.13649874600638 rpy=3.14159265358979 -5.665498452323E-16 -1.5707963267949 -> xyz=0.626 0 -0.126 rpy=2.4344E-17 -2.6448E-17 -1.5708
- joint joint_4: origin xyz=0.0715000000000143 0 0.0860012539936202 rpy=3.14159265358979 1.5707963267949 0 -> xyz=-0.5305 0 0 rpy=1.6474 1.5708 1.6474
- joint joint_5: axis -1 0 0 -> 0 0 -1; origin xyz=0.0434999999994695 0 -0.459000000267993 rpy=-1.5707963267949 0 0 -> xyz=0.091 0 0 rpy=0 1.5708 0
- joint joint_6: axis 0 0 1 -> 1 0 0; origin xyz=0.0474999999995303 0 0.104999999999948 rpy=3.14159265358979 0 1.5707963267949 -> xyz=0.122 0 0 rpy=2.9386E-15 5.7152E-17 1.15E-16

File: hsr_description/urdf/hsr_br609_with_gripper_kinect.xacro (robot description, xacro)
@@ -1,13 +1,13 @@
 <?xml version="1.0"?>
 <robot
-  name="hsr_jr603" xmlns:xacro="http://www.ros.org/wiki/xacro">
-<xacro:include filename="$(find hsr_description)/urdf/hsr_jr603.urdf" />
+  name="hsr_br609" xmlns:xacro="http://www.ros.org/wiki/xacro">
+<xacro:include filename="$(find hsr_description)/urdf/hsr_br609.urdf" />
   <joint name="gripper_robot_joint" type="fixed">
       <parent link="link6" />
       <child link="gripper_base_link" />
-      <origin xyz="0.0 0.0 0.0" rpy="0 0 0" />
+      <origin xyz="0.0 0.0 0.0" rpy="0 1.5708 0" />
   </joint>
   <joint name="pick_gripper_joint" type="fixed">
-     <origin xyz="-0.0115 0.0 0.15" rpy="0 0 0" />
+     <origin xyz="-0.0115 0.0 0.15" rpy="0 -1.5708 1.5708" />
      <axis xyz="0 0 1"/>
      <parent link="gripper_base_link" />
