Commit message: jr603抓取问题修复

File: hsr_description/urdf/hsr_jr603_with_gripper.xacro (robot description, xacro)
@@ -9,5 +9,5 @@
   </joint>
   <joint name="pick_gripper_joint" type="fixed">
-     <origin xyz="-0.0115 0.0 0.15" rpy="0 -1.5708 1.5708" />
+     <origin xyz="0.0 0.0 0.18" rpy="0 -1.5708 1.5708" />
      <axis xyz="0 0 1"/>
      <parent link="gripper_base_link" />

File: hsr_description/urdf/hsr_jr603_with_gripper_kinect.xacro (robot description, xacro)
@@ -2,17 +2,5 @@
 <robot
   name="hsr_jr603" xmlns:xacro="http://www.ros.org/wiki/xacro">
-<xacro:include filename="$(find hsr_description)/urdf/hsr_jr603.urdf" />
-  <joint name="gripper_robot_joint" type="fixed">
-      <parent link="link6" />
-      <child link="gripper_base_link" />
-      <origin xyz="0.0 0.0 0.0" rpy="0 0 0" />
-  </joint>
-  <joint name="pick_gripper_joint" type="fixed">
-     <origin xyz="-0.0115 0.0 0.15" rpy="0 0 0" />
-     <axis xyz="0 0 1"/>
-     <parent link="gripper_base_link" />
-     <child link="pick_gripper_link" />
-  </joint>
-<xacro:include filename="$(find hsr_description)/urdf/hsr_newtran_gripper.xacro.xml" />
+<xacro:include filename="$(find hsr_description)/urdf/hsr_jr603_with_gripper.xacro" />
 <xacro:include filename="$(find hsr_description)/urdf/hsr_kinect.xacro.xml" />
 </robot>
