Commit message: add eye in hand urdf and launch file

File: hsr_description/urdf/hsr_br606_with_kinect_on_hand.xacro (robot description, xacro)
@@ -18,6 +18,6 @@
   <joint name="camera_joint" type="fixed">
     <axis xyz="0 0 0" />
-    <origin xyz="0.8 0 1.5" rpy="0 1.57 0"/>
-    <parent link="base_link"/>
+    <origin xyz="0 0 -0.05" rpy="0 -1.57 0"/>
+    <parent link="pick_gripper_link"/>
     <child link="camera_link"/>
   </joint>
