Commit message: fixed some bug

File: hsr_description/urdf/hsr_br606.urdf (robot description, URDF)
Before this commit: robot hsr_br606, 8 links, 7 joints
Joints:
- joint fixed: origin (none) -> xyz=0 0 0.4 rpy=0 0 0

Commit message: 合并开发仓库和发布仓库，修复已知BUG

File: hsr_description/urdf/hsr_br606.urdf (robot description, URDF)
Before this commit: robot hsr_br606, 8 links, 7 joints
Joints:
- joint fixed: origin xyz=0 0 0.4 rpy=0 0 0 -> (none)
- joint joint1: limit lower=-3.141596 upper=3.141596 effort=28.0 velocity=3.2 -> lower=-2.71415 upper=2.71415 effort=28.0 velocity=3.2; origin xyz=0 0 0 rpy=1.5707963267949 -1.5707963267949 0 -> xyz=0 0 0 rpy=-1.5707963267949 -1.5707963267949 0
- joint joint2: limit lower=-3.141596 upper=3.141596 effort=28.0 velocity=3.2 -> lower=-3.1 upper=0 effort=28.0 velocity=3.2
- joint joint3: limit lower=-3.141596 upper=3.141596 effort=28.0 velocity=3.2 -> lower=-0.63 upper=3.4 effort=28.0 velocity=3.2
- joint joint4: limit lower=-3.141596 upper=3.141596 effort=28.0 velocity=3.2 -> lower=-1.57 upper=1.57 effort=28.0 velocity=3.2
- joint joint5: limit lower=-3.141596 upper=3.141596 effort=28.0 velocity=3.2 -> lower=-1.68 upper=1.68 effort=28.0 velocity=3.2
- joint joint6: limit lower=-3.141596 upper=3.141596 effort=28.0 velocity=3.2 -> lower=-4.5 upper=4.5 effort=28.0 velocity=3.2

Commit message: 修复ROS-I与机械臂URDF关节名不一致的问题

File: hsr_description/urdf/hsr_br606.urdf (robot description, URDF)
Before this commit: robot hsr_br606, 8 links, 7 joints
Joints:
- removed joint joint1
- removed joint joint2
- removed joint joint3
- removed joint joint4
- removed joint joint5
- removed joint joint6
- added joint joint_1: type revolute, parent base_link, child link1, origin xyz=0 0 0 rpy=-1.5707963267949 -1.5707963267949 0, axis 1 0 0, limit lower=-2.71415 upper=2.71415 effort=28.0 velocity=3.2
- added joint joint_2: type revolute, parent link1, child link2, origin xyz=0 0 -0.0965 rpy=-2.60414512664787E-19 2.50218939158031E-21 1.57079635078175, axis 0 0 1, limit lower=-3.1 upper=0 effort=28.0 velocity=3.2
- added joint joint_3: type revolute, parent link2, child link3, origin xyz=0.725999999928 0 -0.1245 rpy=-2.61618022719008E-33 -1.8705490199458E-25 -1.57079631299268, axis 0 0 1, limit lower=-0.63 upper=3.4 effort=28.0 velocity=3.2
- added joint joint_4: type revolute, parent link3, child link4, origin xyz=-0.630499999499992 0 0 rpy=0 1.5707963267949 0, axis 0 0 -0.999999999999999, limit lower=-1.57 upper=1.57 effort=28.0 velocity=3.2
- added joint joint_5: type revolute, parent link4, child link5, origin xyz=0.091 0 0 rpy=0 1.5708 0, axis 0 0 -1, limit lower=-1.68 upper=1.68 effort=28.0 velocity=3.2
- added joint joint_6: type revolute, parent link5, child link6, origin xyz=0.122 0 0 rpy=1.4901E-08 1.5708 0, axis 0 0 1, limit lower=-4.5 upper=4.5 effort=28.0 velocity=3.2

File: hsr_description/urdf/hsr_br609.urdf (robot description, URDF)
Before this commit: robot hsr_br609, 8 links, 7 joints
Joints:
- removed joint joint1
- removed joint joint2
- removed joint joint3
- removed joint joint4
- removed joint joint5
- removed joint joint6
- added joint joint_1: type continuous, parent base_link, child link1, origin xyz=0 0 0.2755 rpy=-1.5708 -6.123E-17 -1.5708, axis 0 -1 0
- added joint joint_2: type continuous, parent link1, child link2, origin xyz=0 -0.145 0 rpy=-1.5707963267949 -1.22460635382238E-16 1.5707963267949, axis 0 0 -1
- added joint joint_3: type continuous, parent link2, child link3, origin xyz=-0.625999999928 0 -0.13649874600638 rpy=3.14159265358979 -5.665498452323E-16 -1.5707963267949, axis 0 0 1
- added joint joint_4: type continuous, parent link3, child link4, origin xyz=0.0715000000000143 0 0.0860012539936202 rpy=3.14159265358979 1.5707963267949 0, axis 0 0 -1
- added joint joint_5: type continuous, parent link4, child link5, origin xyz=0.0434999999994695 0 -0.459000000267993 rpy=-1.5707963267949 0 0, axis -1 0 0
- added joint joint_6: type continuous, parent link5, child link6, origin xyz=0.0474999999995303 0 0.104999999999948 rpy=3.14159265358979 0 1.5707963267949, axis 0 0 1

File: hsr_description/urdf/hsr_co602.urdf (robot description, URDF)
Before this commit: robot hsr_co602, 8 links, 7 joints
Joints:
- removed joint joint1
- removed joint joint2
- removed joint joint3
- removed joint joint4
- removed joint joint5
- removed joint joint6
- added joint joint_1: type revolute, parent base_link, child link1, origin xyz=0 0 0 rpy=-2.4562E-16 -3.154E-16 9.8608E-32, axis 0 0 1, limit lower=-3.4 upper=3.4 effort=28.0 velocity=3.2
- added joint joint_2: type revolute, parent link1, child link2, origin xyz=0 0.221 0 rpy=-1.5708 3.2234E-16 -9.0966E-30, axis 0 0 1, limit lower=-3.0 upper=0.0 effort=28.0 velocity=3.2
- added joint joint_3: type revolute, parent link2, child link3, origin xyz=0.425 0 0 rpy=6.7185E-17 -3.5791E-18 1.1796E-16, axis 0 0 1, limit lower=1.4 upper=4.0 effort=28.0 velocity=3.2
- added joint joint_4: type revolute, parent link3, child link4, origin xyz=0 0 -0.172 rpy=-1.5707963267949 -6.01453096837983E-18 3.14159265358979, axis 0 0 1, limit lower=-3.0 upper=3.0 effort=28.0 velocity=3.2
- added joint joint_5: type revolute, parent link4, child link5, origin xyz=0 -0.1605 0.375 rpy=-1.5708 -6.9389E-18 2.9856E-17, axis 0 0 -1, limit lower=-1.9 upper=1.9 effort=28.0 velocity=3.2
- added joint joint_6: type revolute, parent link5, child link6, origin xyz=0 -0.1615 0 rpy=1.5708 -9.3415E-18 -4.21E-18, axis 0 0 1, limit lower=-6 upper=6 effort=28.0 velocity=3.2

File: hsr_description/urdf/hsr_jr605.urdf (robot description, URDF)
Before this commit: robot hsr_jr605, 7 links, 6 joints
Joints:
- removed joint joint1
- removed joint joint2
- removed joint joint3
- removed joint joint4
- removed joint joint5
- removed joint joint6
- added joint joint_1: type revolute, parent base_link, child link1, origin xyz=0 0 0.3535 rpy=0 0 0, axis 0 0 1, limit lower=-3.4907 upper=3.4907 effort=0 velocity=0
- added joint joint_2: type revolute, parent link1, child link2, origin xyz=0 0 0 rpy=-1.5708 0 9.8233E-20, axis 0 0 1, limit lower=-3.1416 upper=0.0175 effort=0 velocity=0
- added joint joint_3: type revolute, parent link2, child link3, origin xyz=0.36 0 0 rpy=-1.2635E-17 5.072E-19 4.9915E-36, axis 0 0 1, limit lower=1.3963 upper=4.1888 effort=0 velocity=0
- added joint joint_4: type revolute, parent link3, child link4, origin xyz=-0.09 0 0 rpy=1.5708 0 0, axis 0 0 -1, limit lower=-3.1416 upper=3.1416 effort=0 velocity=0
- added joint joint_5: type revolute, parent link4, child link5, origin xyz=0 0 0.3765 rpy=-1.5708 -1.3878E-17 -4.4702E-16, axis 0 0 1, limit lower=-2.0071 upper=2.0071 effort=0 velocity=0
- added joint joint_6: type revolute, parent link5, child link6, origin xyz=0 -0.119 0 rpy=1.5708 0.042291 1.1639E-17, axis 0 0 -1, limit lower=-6.2832 upper=6.2832 effort=0 velocity=0

Commit message: fixed br606 urdf inertia and limit bug

File: hsr_description/urdf/hsr_br606.urdf (robot description, URDF)
Before this commit: robot hsr_br606, 8 links, 7 joints
Links:
- link base_link: mass 10.9537086254326 -> 10.954
- link link1: mass 4.59272942117021 -> 4.59276430213053
- link link2: mass 6.56007074220098 -> 6.56009345873244
- link link3: mass 1.11116815174246 -> 1.11115013215577
- link link4: mass 3.18597528812718 -> 3.18597657698263
- link link5: mass 0.8684 -> 0.868404071249388
- link link6: mass 0.027077 -> 0.0270769176823693
Joints:
- joint fixed: origin (none) -> xyz=0 0 1 rpy=0 0 0

Commit message: br606零点更新

File: hsr_description/urdf/hsr_br606.urdf (robot description, URDF)
Before this commit: robot hsr_br606, 8 links, 7 joints
Joints:
- joint joint_3: limit lower=-0.63 upper=3.4 effort=28.0 velocity=3.2 -> lower=2.3 upper=7 effort=28.0 velocity=3.2; origin xyz=0.725999999928 0 -0.1245 rpy=-2.61618022719008E-33 -1.8705490199458E-25 -1.57079631299268 -> xyz=0.725999999928 0 -0.1245 rpy=-2.61618022719008E-33 -1.8705490199458E-25 1.57079631299268

File: hsr_description/urdf/hsr_br606_with_eye_hand_gripper.xacro (robot description, xacro)
@@ -6,5 +6,5 @@
       <parent link="link6" />
       <child link="gripper_base_link" />
-      <origin xyz="0.0 0.0 0.0" rpy="0 0 0.7853981633975" />
+      <origin xyz="0.0 0.0 0.0" rpy="0 0 3.14" />
   </joint>
   <joint name="pick_gripper_joint" type="fixed">
@@ -14,11 +14,4 @@
      <child link="pick_gripper_link" />
   </joint>
-<xacro:include filename="$(find hsr_description)/urdf/hsr_gripper.xacro.xml" />
-<xacro:include filename="$(find hsr_description)/urdf/hsr_kinect.xacro.xml" />
-  <joint name="camera_joint" type="fixed">
-    <axis xyz="0 0 0" />
-    <origin xyz="0.8 0 1.5" rpy="0 1.57 0"/>
-    <parent link="base_link"/>
-    <child link="camera_link"/>
-  </joint>
+<xacro:include filename="$(find hsr_description)/urdf/eye_hand_gripper.xacro.xml" />
 </robot>
