Commit message: add br606 moveit config and udpade urdf

File: hsr_description/urdf/hsr_br606_with_eye_hand_gripper.xacro (robot description, xacro)
@@ -1,17 +1,17 @@
 <?xml version="1.0"?>
 <robot
-  name="hsr_jr603" xmlns:xacro="http://www.ros.org/wiki/xacro">
-<xacro:include filename="$(find hsr_description)/urdf/hsr_jr603.urdf" />
+  name="hsr_br606" xmlns:xacro="http://www.ros.org/wiki/xacro">
+<xacro:include filename="$(find hsr_description)/urdf/hsr_br606.urdf" />
   <joint name="gripper_robot_joint" type="fixed">
       <parent link="link6" />
       <child link="gripper_base_link" />
-      <origin xyz="0.0 0.0 0.0" rpy="0 0 0" />
+      <origin xyz="0.0 0.0 0.0" rpy="0 0 3.14" />
   </joint>
   <joint name="pick_gripper_joint" type="fixed">
-     <origin xyz="0.0 0.0 0.18" rpy="0 -1.5708 1.5708" />
+     <origin xyz="-0.0115 0.0 0.15" rpy="0 -1.5708 1.5708" />
      <axis xyz="0 0 1"/>
      <parent link="gripper_base_link" />
      <child link="pick_gripper_link" />
   </joint>
-<xacro:include filename="$(find hsr_description)/urdf/hsr_newtran_gripper.xacro.xml" />
+<xacro:include filename="$(find hsr_description)/urdf/eye_hand_gripper.xacro.xml" />
 </robot>

File: hsr_description/urdf/hsr_br606_with_gripper_kinect.xacro (robot description, xacro)
@@ -6,5 +6,5 @@
       <parent link="link6" />
       <child link="gripper_base_link" />
-      <origin xyz="0.0 0.0 0.0" rpy="0 0 0" />
+      <origin xyz="0.0 0.0 0.0" rpy="0 0 0.7853981633975" />
   </joint>
   <joint name="pick_gripper_joint" type="fixed">
@@ -16,3 +16,9 @@
 <xacro:include filename="$(find hsr_description)/urdf/hsr_gripper.xacro.xml" />
 <xacro:include filename="$(find hsr_description)/urdf/hsr_kinect.xacro.xml" />
+  <joint name="camera_joint" type="fixed">
+    <axis xyz="0 0 0" />
+    <origin xyz="0.8 0 1.5" rpy="0 1.57 0"/>
+    <parent link="base_link"/>
+    <child link="camera_link"/>
+  </joint>
 </robot>

File: hsr_description/urdf/hsr_br606_with_kinect_on_hand.xacro (robot description, xacro)
@@ -6,5 +6,5 @@
       <parent link="link6" />
       <child link="gripper_base_link" />
-      <origin xyz="0.0 0.0 0.0" rpy="0 0 3.14" />
+      <origin xyz="0.0 0.0 0.0" rpy="0 0 0" />
   </joint>
   <joint name="pick_gripper_joint" type="fixed">
@@ -14,5 +14,11 @@
      <child link="pick_gripper_link" />
   </joint>
-<xacro:include filename="$(find hsr_description)/urdf/eye_hand_gripper.xacro.xml" />
+<xacro:include filename="$(find hsr_description)/urdf/hsr_gripper.xacro.xml" />
 <xacro:include filename="$(find hsr_description)/urdf/hsr_kinect.xacro.xml" />
+  <joint name="camera_joint" type="fixed">
+    <axis xyz="0 0 0" />
+    <origin xyz="0 0 -0.05" rpy="0 -1.57 0"/>
+    <parent link="pick_gripper_link"/>
+    <child link="camera_link"/>
+  </joint>
 </robot>
