Commit message: Add co602a driver, Updata ros-i drvier

File: hsr_description/urdf/hsr_co602a_test.urdf (robot description, URDF)
Before this commit: robot hsr_co602a, 7 links, 6 joints
Links:
- removed link robot_base_link
- added link link_base, mass 4.8818; collision mesh filename=package://hsr_description/meshes/co602a/link_base.STL; visual mesh filename=package://hsr_description/meshes/co602a/link_base.STL
Joints:
- joint joint_1: parent robot_base_link -> link_base
