Commit message: 1，删除无用的launch文件 2，解决RVIZ配置文件路径不生效的问题 3，解决每次都需要设置joint_name的问题

File: hsr_description/urdf/hsr_co602a.urdf (robot description, URDF)
Before this commit: robot hsr_co602a, 7 links, 6 joints
Links:
- removed link robot_base_link
- added link base_link, mass 4.8818; collision mesh filename=package://hsr_description/meshes/co602a/base_link.STL; visual mesh filename=package://hsr_description/meshes/co602a/base_link.STL
- added link world
Joints:
- added joint fixed: type fixed, parent world, child base_link, origin xyz=0 0 1 rpy=0 0 0
- joint joint_1: parent robot_base_link -> base_link
