Commit message: 1，修复hsr_moveit_api中的base_api一些已知问题 2，修复co

File: hsr_description/urdf/hsr_co602_with_eyeonhand_gripper.xacro (robot description, xacro)
@@ -9,5 +9,5 @@
   </joint>
   <joint name="pick_gripper_joint" type="fixed">
-     <origin xyz="-0.0115 0.0 0.15" rpy="0 -1.5708 1.5708" />
+     <origin xyz="0 0.0 0.18" rpy="0 -1.5708 1.5708" />
      <axis xyz="0 0 1"/>
      <parent link="gripper_base_link" />
