Commit message: 五指夹爪和双臂的抓取代码块

File: hsr_description/urdf/hsr_co605-test.urdf (robot description, URDF)
Before this commit: robot hsr_co605, 15 links, 14 joints
Links:
- link R_link1: mass 2.2858 -> 4.9043; geometry collision mesh filename=package://hsr_co602a_gaihou/meshes/Link1.STL; visual mesh filename=package://hsr_co602a_gaihou/meshes/Link1.STL
- link R_link2: mass 3.9796 -> 6.5305; geometry collision mesh filename=package://hsr_co602a_gaihou/meshes/Link2.STL; visual mesh filename=package://hsr_co602a_gaihou/meshes/Link2.STL
- link R_link3: mass 2.3017 -> 2.3223; geometry collision mesh filename=package://hsr_co602a_gaihou/meshes/Link3.STL; visual mesh filename=package://hsr_co602a_gaihou/meshes/Link3.STL
- link R_link4: mass 1.1696 -> 1.2629; geometry collision mesh filename=package://hsr_co602a_gaihou/meshes/Link4.STL; visual mesh filename=package://hsr_co602a_gaihou/meshes/Link4.STL
- link R_link5: mass 1.4115 -> 1.1452; geometry collision mesh filename=package://hsr_co602a_gaihou/meshes/Link5.STL; visual mesh filename=package://hsr_co602a_gaihou/meshes/Link5.STL
- link R_link6: mass 0.30888 -> 0.20458; geometry collision mesh filename=package://hsr_co602a_gaihou/meshes/Link6.STL; visual mesh filename=package://hsr_co602a_gaihou/meshes/Link6.STL
- link base_link2: mass 3.5836 -> 4.8818; geometry collision mesh filename=package://hsr_co602a_gaihou/meshes/base_link.STL; visual mesh filename=package://hsr_co602a_gaihou/meshes/base_link.STL
Joints:
- joint R_joint_1: origin xyz=0 0 0.3215 rpy=-3.1416 5.9903E-29 -1.4937E-16 -> xyz=0 0 0.3517 rpy=3.1416 0 -8.3267E-17
- joint R_joint_3: origin xyz=0 -0.4 0 rpy=-7.0321E-15 1.0327E-14 -1.5708 -> xyz=0 -0.40061 0 rpy=-3.688E-17 1.4367E-17 -1.5708
- joint R_joint_4: limit lower=-3.0 upper=3.0 effort=28 velocity=3.2 -> lower=-1.0 upper=3.0 effort=28 velocity=3.2; origin xyz=0 0 0 rpy=1.5708 1.5708 0 -> xyz=0 -0.0023254 0 rpy=1.2216 1.5708 -0.34916
- joint R_joint_5: origin xyz=0 0 0.4 rpy=-1.5708 -3.2281E-16 1.5708 -> xyz=0 0 0.39859 rpy=-1.5708 -1.4529E-17 1.5708
- joint R_joint_6: origin xyz=0 -0.205 0 rpy=-1.5708 2.7756E-17 -3.1416 -> xyz=0 -0.20056 0 rpy=-1.5708 2.4478E-17 -3.1416
- joint fixed2: origin xyz=0 1 1 rpy=0 0 0 -> xyz=0.025 1 1 rpy=0 0 0
